Commit message: tests: Friction and surface tests

File: qcar_description/urdf/qcar_ros2.urdf.xacro (robot description, xacro)
@@ -519,18 +519,88 @@
     </gazebo>
     <gazebo reference="right_front_wheel">
-      <mu1>100.0</mu1>
-      <mu2>100.0</mu2>
+      <collision>
+        <surface>
+          <friction>
+            <ode>
+              <mu>1.0</mu>
+              <mu2>1.0</mu2>
+              <fdir1>0 0 1</fdir1>
+            </ode>
+          </friction>
+          <contact>
+            <ode>
+              <kp>1000000.0</kp>
+              <kd>100.0</kd>
+              <max_vel>0.1</max_vel>
+              <min_depth>0.001</min_depth>
+            </ode>
+          </contact>
+        </surface>
+      </collision>
     </gazebo>
     <gazebo reference="left_front_wheel">
-      <mu1>100.0</mu1>
-      <mu2>100.0</mu2>
+      <collision>
+        <surface>
+          <friction>
+            <ode>
+              <mu>1.0</mu>
+              <mu2>1.0</mu2>
+              <fdir1>0 0 1</fdir1>
+            </ode>
+          </friction>
+          <contact>
+            <ode>
+              <kp>1000000.0</kp>
+              <kd>100.0</kd>
+              <max_vel>0.1</max_vel>
+              <min_depth>0.001</min_depth>
+            </ode>
+          </contact>
+        </surface>
+      </collision>
     </gazebo>
     <gazebo reference="right_rear_wheel">
-      <mu1>100.0</mu1>
-      <mu2>100.0</mu2>
+      <collision>
+        <surface>
+          <friction>
+            <ode>
+              <mu>1.0</mu>
+              <mu2>1.0</mu2>
+              <fdir1>0 0 1</fdir1>
+            </ode>
+          </friction>
+          <contact>
+            <ode>
+              <kp>1000000.0</kp>
+              <kd>100.0</kd>
+              <max_vel>0.1</max_vel>
+              <min_depth>0.001</min_depth>
+            </ode>
+          </contact>
+        </surface>
+      </collision>
     </gazebo>
     <gazebo reference="left_rear_wheel">
-      <mu1>100.0</mu1>
-      <mu2>100.0</mu2>
+      <collision>
+        <surface>
+          <friction>
+            <ode>
+              <mu>1.0</mu>
+              <mu2>1.0</mu2>
+              <fdir1>0 0 1</fdir1>
+            </ode>
+          </friction>
+          <contact>
+            <ode>
+              <kp>1000000.0</kp>
+              <kd>100.0</kd>
+              <max_vel>0.1</max_vel>
+              <min_depth>0.001</min_depth>
+            </ode>
+          </contact>
+        </surface>
+      </collision>
+      <!-- <mu1>100.0</mu1>
+      <mu2>100.0</mu2> -->
     </gazebo>
     <!--<gazebo>
