Commit message: added: scan and odometry to the gazebo implementation of the qcar

File: qcar_description/urdf/qcar.gazebo.xacro (robot description, xacro)
@@ -1,324 +1,369 @@
 <?xml version="1.0"?>
 <robot name="QCar" xmlns:xacro="http://www.ros.org/wiki/xacro">
-  <xacro:property name="max_steering_angle" value="0.3"/>
-  <xacro:property name="axle_vel_limit" value="244.8696"/>
-  <link name="camera_rgb_optical_link"/>
-  <joint name="camera_rgb_optical_joint" type="fixed">
-    <!-- these values have to be these values otherwise the gazebo camera
-        image won't be aligned properly with the frame it is supposedly
-        originating from -->
-    <origin xyz="0 0 0" rpy="${-pi/2} 0 ${-pi/2}"/>
-    <parent link="camera_rgb"/>
-    <child link="camera_rgb_optical_link"/>
-  </joint>
-<!-- Define all the computer vision sernsor properties -->
-	<gazebo reference="camera_rgb">
-    <!-- <material>Gazebo/Green</material> -->
-    <sensor type="camera" name="intelrealsense_rgb">
-      <always_on>1</always_on>
-      <update_rate>60.0</update_rate>
-      <visualize>true</visualize>
-      <topic>qcar/rgb/image_raw</topic>
-      <camera name="rgb">
-        <horizontal_fov>1.21126</horizontal_fov>
-        <image>
-            <width>640</width>
-            <height>480</height>
-            <format>R8G8B8</format>
-        </image>
-        <clip>
-            <near>0.02</near>
-            <far>300</far>
-        </clip>
-        <noise>
-            <type>gaussian</type>
-            <mean>0.0</mean>
-            <stddev>0.001</stddev>
-        </noise>
-        <distortion>
-          <k1>0.0</k1>
-          <k2>0.0</k2>
-          <k3>0.0</k3>
-          <p1>0.0</p1>
-          <p2>0.0</p2>
-        </distortion>
-        <optical_frame_id>camera_rgb_optical_link</optical_frame_id>
-        <camera_info_topic>qcar/rgb/camera_info</camera_info_topic>
-      </camera>
-    </sensor>
-  </gazebo>
-  <link name="camera_csi_front_optical_link"/>
-  <joint name="camera_csi_front_optical_joint" type="fixed">
-    <!-- these values have to be these values otherwise the gazebo camera
-        image won't be aligned properly with the frame it is supposedly
-        originating from -->
-    <origin xyz="0 0 0" rpy="${-pi/2} 0 ${-pi/2}"/>
-    <parent link="camera_csi_front"/>
-    <child link="camera_csi_front_optical_link"/>
-  </joint>
-<!-- Define all the computer vision sernsor properties -->
-	<gazebo reference="camera_csi_front">
-    <!-- <material>Gazebo/Green</material> -->
-    <sensor type="camera" name="csi_front">
-      <always_on>1</always_on>
-      <update_rate>60.0</update_rate>
-      <visualize>true</visualize>
-      <topic>qcar/csi_front/image_raw</topic>
-      <camera name="front">
-        <horizontal_fov>2.79253</horizontal_fov>
-        <image>
-            <width>1280</width>
-            <height>640</height>
-            <format>R8G8B8</format>
-        </image>
-        <clip>
-            <near>0.02</near>
-            <far>300</far>
-        </clip>
-        <noise>
-            <type>gaussian</type>
-            <mean>0.0</mean>
-            <stddev>0.001</stddev>
-        </noise>
-        <distortion>
-          <k1>-0.264598808</k1>
-          <k2>0.0156281135</k2>
-          <k3>0.0822019378</k3>
-          <p1>0.0000652954</p1>
-          <p2>0.0053984313</p2>
-        </distortion>
-        <optical_frame_id>camera_csi_front_optical_link</optical_frame_id>
-        <camera_info_topic>qcar/csi_front/camera_info</camera_info_topic>
-      </camera>
-    </sensor>
-  </gazebo>
-  <link name="camera_csi_right_optical_link"/>
-  <joint name="camera_csi_right_optical_joint" type="fixed">
-    <!-- these values have to be these values otherwise the gazebo camera
-        image won't be aligned properly with the frame it is supposedly
-        originating from -->
-    <origin xyz="0 0 0" rpy="${-pi/2} 0 ${-pi/2}"/>
-    <parent link="camera_csi_right"/>
-    <child link="camera_csi_right_optical_link"/>
-  </joint>
-<!-- Define all the computer vision sernsor properties -->
-	<gazebo reference="camera_csi_right">
-    <!-- <material>Gazebo/Green</material> -->
-    <sensor type="camera" name="csi_right">
-      <always_on>1</always_on>
-      <update_rate>60.0</update_rate>
-      <visualize>true</visualize>
-      <topic>qcar/csi_right/image_raw</topic>
-      <camera name="right">
-        <horizontal_fov>2.79253</horizontal_fov>
-        <image>
-            <width>1280</width>
-            <height>640</height>
-            <format>R8G8B8</format>
-        </image>
-        <clip>
-            <near>0.02</near>
-            <far>300</far>
-        </clip>
-        <noise>
-            <type>gaussian</type>
-            <mean>0.0</mean>
-            <stddev>0.001</stddev>
-        </noise>
-        <distortion>
-          <k1>-0.264598808</k1>
-          <k2>0.0156281135</k2>
-          <k3>0.0822019378</k3>
-          <p1>0.0000652954</p1>
-          <p2>0.0053984313</p2>
-        </distortion>
-        <optical_frame_id>camera_csi_right_optical_link</optical_frame_id>
-        <camera_info_topic>qcar/csi_right/camera_info</camera_info_topic>
-      </camera>
-    </sensor>
-  </gazebo>
-  <link name="camera_csi_left_optical_link"/>
-  <joint name="camera_csi_left_optical_joint" type="fixed">
-    <!-- these values have to be these values otherwise the gazebo camera
-        image won't be aligned properly with the frame it is supposedly
-        originating from -->
-    <origin xyz="0 0 0" rpy="${-pi/2} 0 ${-pi/2}"/>
-    <parent link="camera_csi_left"/>
-    <child link="camera_csi_left_optical_link"/>
-  </joint>
-<!-- Define all the computer vision sernsor properties -->
-	<gazebo reference="camera_csi_left">
-    <!-- <material>Gazebo/Green</material> -->
-    <sensor type="camera" name="csi_left">
-      <always_on>1</always_on>
-      <update_rate>60.0</update_rate>
-      <visualize>true</visualize>
-      <topic>qcar/csi_left/image_raw</topic>
-      <camera name="front">
-        <horizontal_fov>2.79253</horizontal_fov>
-        <image>
-            <width>1280</width>
-            <height>640</height>
-            <format>R8G8B8</format>
-        </image>
-        <clip>
-            <near>0.02</near>
-            <far>300</far>
-        </clip>
-        <noise>
-            <type>gaussian</type>
-            <mean>0.0</mean>
-            <stddev>0.001</stddev>
-        </noise>
-        <distortion>
-          <k1>-0.264598808</k1>
-          <k2>0.0156281135</k2>
-          <k3>0.0822019378</k3>
-          <p1>0.0000652954</p1>
-          <p2>0.0053984313</p2>
-        </distortion>
-        <optical_frame_id>camera_csi_left_optical_link</optical_frame_id>
-        <camera_info_topic>qcar/csi_left/camera_info</camera_info_topic>
-      </camera>
-    </sensor>
-  </gazebo>
-  <link name="camera_csi_back_optical_link"/>
-  <joint name="camera_csi_back_optical_joint" type="fixed">
-    <!-- these values have to be these values otherwise the gazebo camera
-        image won't be aligned properly with the frame it is supposedly
-        originating from -->
-    <origin xyz="0 0 0" rpy="${-pi/2} 0 ${-pi/2}"/>
-    <parent link="camera_csi_back"/>
-    <child link="camera_csi_back_optical_link"/>
-  </joint>
-<!-- Define all the computer vision sernsor properties -->
-	<gazebo reference="camera_csi_back">
-    <!-- <material>Gazebo/Green</material> -->
-    <sensor type="camera" name="csi_back">
-      <always_on>1</always_on>
-      <update_rate>60.0</update_rate>
-      <visualize>true</visualize>
-      <topic>qcar/csi_back/image_raw</topic>
-      <camera name="front">
-        <horizontal_fov>2.79253</horizontal_fov>
-        <image>
-            <width>1280</width>
-            <height>640</height>
-            <format>R8G8B8</format>
-        </image>
-        <clip>
-            <near>0.02</near>
-            <far>300</far>
-        </clip>
-        <noise>
-            <type>gaussian</type>
-            <mean>0.0</mean>
-            <stddev>0.001</stddev>
-        </noise>
-        <distortion>
-          <k1>-0.264598808</k1>
-          <k2>0.0156281135</k2>
-          <k3>0.0822019378</k3>
-          <p1>0.0000652954</p1>
-          <p2>0.0053984313</p2>
-        </distortion>
-        <optical_frame_id>camera_csi_back_optical_link</optical_frame_id>
-        <camera_info_topic>qcar/csi_back/camera_info</camera_info_topic>
-      </camera>
-    </sensor>
-  </gazebo>
-  <!-- Gazebo Parameters -->
-    <gazebo reference="base">
-      <mu1>0.0001</mu1>
-      <mu2>0.0001</mu2>
-    </gazebo>
-    <gazebo reference="right_front_wheel">
-      <mu1>100.0</mu1>
-      <mu2>100.0</mu2>
-    </gazebo>
-    <gazebo reference="left_front_wheel">
-      <mu1>100.0</mu1>
-      <mu2>100.0</mu2>
-    </gazebo>
-    <gazebo reference="right_rear_wheel">
-      <mu1>100.0</mu1>
-      <mu2>100.0</mu2>
-    </gazebo>
-    <gazebo reference="left_rear_wheel">
-      <mu1>100.0</mu1>
-      <mu2>100.0</mu2>
-    </gazebo>
-  <!-- Gazebo Control -->
-  <ros2_control name="control" type="system">
-    <hardware>
-      <plugin>gz_ros2_control/GazeboSimSystem</plugin>
-    </hardware>
-    <joint name="left_steering_joint">
-      <command_interface name="position">
-        <param name="min">${-max_steering_angle}</param>
-        <param name="max">${max_steering_angle}</param>
-      </command_interface>
-      <state_interface name="position"/>
-      <state_interface name="velocity"/>
-      <state_interface name="effort"/>
-    </joint>
-    <joint name="right_steering_joint">
-      <param name="mimic">left_steering_joint</param> <!-- Command this joint -->
-      <param name="multiplier">1</param> <!-- Move in the opposite direction -->
-      <state_interface name="position"/>
-      <state_interface name="velocity"/>
-      <state_interface name="effort"/>
-    </joint>
-    <joint name="right_front_axle">
-      <command_interface name="velocity">
-        <param name="min">${-axle_vel_limit}</param>
-        <param name="max">${axle_vel_limit}</param>
-      </command_interface>
-      <state_interface name="position"/>
-      <state_interface name="velocity"/>
-      <state_interface name="effort"/>
-    </joint>
-    <joint name="left_front_axle">
-      <param name="mimic">right_front_axle</param> <!-- Command this joint -->
-      <param name="multiplier">-1</param> <!-- Move in the opposite direction -->
-      <state_interface name="position"/>
-      <state_interface name="velocity"/>
-      <state_interface name="effort"/>
-    </joint>
-    <joint name="right_rear_axle">
-      <command_interface name="velocity">
-        <param name="min">${-axle_vel_limit}</param>
-        <param name="max">${axle_vel_limit}</param>
-      </command_interface>
-      <state_interface name="position"/>
-      <state_interface name="velocity"/>
-      <state_interface name="effort"/>
-    </joint>
-    <joint name="left_rear_axle">
-      <command_interface name="velocity">
-        <param name="min">${-axle_vel_limit}</param>
-        <param name="max">${axle_vel_limit}</param>
-      </command_interface>
-      <state_interface name="position"/>
-      <state_interface name="velocity"/>
-      <state_interface name="effort"/>
-    </joint>
-  </ros2_control>
-  <gazebo>
-    <plugin filename="gz-sim-joint-state-publisher-system" name="gz::sim::systems::JointStatePublisher">
-      <topic>joint_states</topic>
-      <joint_name>left_steering_joint</joint_name>
-      <joint_name>right_steering_joint</joint_name>
-      <joint_name>left_front_axle</joint_name>
-      <joint_name>right_front_axle</joint_name>
-      <joint_name>left_rear_axle</joint_name>
-      <joint_name>right_rear_axle</joint_name>
-    </plugin>
-    <plugin filename="gz_ros2_control-system" name="gz_ros2_control::GazeboSimROS2ControlPlugin">
-      <parameters>$(find qcar_gazebo)/config/gz_ros2_control.yaml</parameters>
-    </plugin>
-    <plugin filename="gz-sim-sensors-system" name="gz::sim::systems::Sensors">
-        <render_engine>ogre2</render_engine>
-    </plugin>
-  </gazebo>
+  <xacro:macro name="qcar_gazebo" params="is_ign">
+    <xacro:property name="max_steering_angle" value="0.3"/>
+    <xacro:property name="axle_vel_limit" value="244.8696"/>
+    <link name="camera_rgb_optical_link"/>
+    <joint name="camera_rgb_optical_joint" type="fixed">
+      <!-- these values have to be these values otherwise the gazebo camera
+          image won't be aligned properly with the frame it is supposedly
+          originating from -->
+      <origin xyz="0.01 0 0" rpy="${-pi/2} 0 ${-pi/2}"/>
+      <parent link="camera_rgb"/>
+      <child link="camera_rgb_optical_link"/>
+    </joint>
+    <!-- Define all the computer vision sernsor properties -->
+    <gazebo reference="camera_rgb">
+      <!-- <material>Gazebo/Green</material> -->
+      <sensor type="camera" name="intelrealsense_rgb">
+        <always_on>1</always_on>
+        <update_rate>60.0</update_rate>
+        <visualize>true</visualize>
+        <topic>qcar/rgb/image_raw</topic>
+        <camera name="rgb">
+          <horizontal_fov>1.21126</horizontal_fov>
+          <image>
+              <width>640</width>
+              <height>480</height>
+              <format>R8G8B8</format>
+          </image>
+          <clip>
+              <near>0.02</near>
+              <far>300</far>
+          </clip>
+          <noise>
+              <type>gaussian</type>
+              <mean>0.0</mean>
+              <stddev>0.001</stddev>
+          </noise>
+          <distortion>
+            <k1>0.0</k1>
+            <k2>0.0</k2>
+            <k3>0.0</k3>
+            <p1>0.0</p1>
+            <p2>0.0</p2>
+          </distortion>
+          <optical_frame_id>camera_rgb_optical_link</optical_frame_id>
+          <camera_info_topic>qcar/rgb/camera_info</camera_info_topic>
+        </camera>
+      </sensor>
+    </gazebo>
+    <link name="camera_csi_front_optical_link"/>
+    <joint name="camera_csi_front_optical_joint" type="fixed">
+      <!-- these values have to be these values otherwise the gazebo camera
+          image won't be aligned properly with the frame it is supposedly
+          originating from -->
+      <origin xyz="0 0 0" rpy="${-pi/2} 0 ${-pi/2}"/>
+      <parent link="camera_csi_front"/>
+      <child link="camera_csi_front_optical_link"/>
+    </joint>
+  <!-- Define all the computer vision sernsor properties -->
+    <gazebo reference="camera_csi_front">
+      <!-- <material>Gazebo/Green</material> -->
+      <sensor type="camera" name="csi_front">
+        <always_on>1</always_on>
+        <update_rate>60.0</update_rate>
+        <visualize>true</visualize>
+        <topic>qcar/csi_front/image_raw</topic>
+        <camera name="front">
+          <horizontal_fov>2.79253</horizontal_fov>
+          <image>
+              <width>1280</width>
+              <height>640</height>
+              <format>R8G8B8</format>
+          </image>
+          <clip>
+              <near>0.02</near>
+              <far>300</far>
+          </clip>
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
File: qcar_description/urdf/qcar_ros2.urdf.xacro (robot description, xacro)
@@ -502,4 +502,25 @@
     </joint>
     <!-- The above is for the wheels and turning etc -->
+    <!-- Gazebo Parameters -->
+    <gazebo reference="base">
+      <mu1>0.0001</mu1>
+      <mu2>0.0001</mu2>
+    </gazebo>
+    <gazebo reference="right_front_wheel">
+      <mu1>100.0</mu1>
+      <mu2>100.0</mu2>
+    </gazebo>
+    <gazebo reference="left_front_wheel">
+      <mu1>100.0</mu1>
+      <mu2>100.0</mu2>
+    </gazebo>
+    <gazebo reference="right_rear_wheel">
+      <mu1>100.0</mu1>
+      <mu2>100.0</mu2>
+    </gazebo>
+    <gazebo reference="left_rear_wheel">
+      <mu1>100.0</mu1>
+      <mu2>100.0</mu2>
+    </gazebo>
     <!--<gazebo>
       <plugin name="gazebo_ros_control" filename="libgazebo_ros_control.so" />

File: qcar_description/urdf/qcar_system.urdf.xacro (robot description, xacro)
@@ -5,11 +5,22 @@
   <xacro:arg name="use_fake_hardware" default="true" />
   <xacro:arg name="fake_sensor_commands" default="false" />
+  <xacro:arg name="is_ign" default="false" />
   <xacro:arg name="prefix" default="" />
   <xacro:include filename="$(find qcar_description)/urdf/qcar_ros2.urdf.xacro" />
   <!-- Import all Gazebo-customization elements, including Gazebo colors -->
   <xacro:include filename="$(find qcar_description)/urdf/qcar.gazebo.xacro" />
+  <!-- Import Rviz colors -->
+  <!-- <xacro:include filename="$(find qcar_description)/urdf/qcar.materials.xacro" /> -->
+  <!-- Import diffbot ros2_control description -->
+  <!-- <xacro:include filename="$(find qcar_description)/ros2_control/qcar_system.ros2_control.xacro" /> -->
+  <!-- Used for fixing robot -->
+  <!-- <link name="world"/> -->
+  <!-- <gazebo reference="world">
+    <static>false</static>
+  </gazebo> -->
   <xacro:QCar parent="world" prefix="$(arg prefix)">
     <origin xyz="0 0 0" rpy="0 0 0" />
   </xacro:QCar>
+  <xacro:qcar_gazebo is_ign="$(arg is_ign)"/>
   <!-- <xacro:QCar_control name="QCar" prefix="$(arg prefix)"/> -->
 </robot>

Commit message: modification: adding imu to the digital twin, work in progress

File: qcar_description/urdf/qcar.gazebo.xacro (robot description, xacro)
@@ -266,4 +266,18 @@
       </sensor>
     </gazebo>
+    <gazebo reference="imu">
+      <sensor name="imu" type="imu">
+        <always_on>1</always_on>
+        <update_rate>60.0</update_rate>
+        <visualize>true</visualize>
+        <topic>imu</topic>
+        <imu>
+          <orientation_reference_frame>
+            <localization>GRAV_UP</localization>
+          </orientation_reference_frame>
+        </imu>
+      <!-- Sensor |camera,ray,imu,magnetometer,gps,force_torque,contact,sonar,rfidtag,rfid| -->
+      </sensor>
+    </gazebo>
     <gazebo>
       <xacro:unless value="${is_ign}">

File: qcar_description/urdf/qcar_ros2.urdf.xacro (robot description, xacro)
@@ -248,4 +248,15 @@
     </joint>
     <link name="camera_csi_left"/>
+    <joint name="imu_joint" type="fixed">
+        <!-- <axis xyz="0 1 0" /> -->
+        <!-- <origin xyz=".2 0 0" rpy="0 0 0"/> -->
+        <!-- ___________________xyz is wrong, need to update_______________________________ -->
+        <!-- <origin rpy="0 0 1.5708" xyz="0.12784 0.052497 0.093029"/> -->
+         <origin rpy="0 0 0" xyz="0.1278 0.0223 0.087229"/>
+        <!-- <origin rpy="0 0 0" xyz="0 0 0"/> -->
+        <parent link="base"/>
+        <child link="imu"/>
+    </joint>
+    <link name="imu"/>
     <!-- <transmission name="body_lidar_tran">
         <type>>transmission_interface/SimpleTransmission</type>
