Commit message: modification:  better simulation results

File: qcar_description/urdf/qcar.gazebo.xacro (robot description, xacro)
@@ -1,5 +1,6 @@
 <?xml version="1.0"?>
 <robot name="QCar" xmlns:xacro="http://www.ros.org/wiki/xacro">
-  <xacro:macro name="qcar_gazebo" params="is_ign">
+  <xacro:macro name="qcar_gazebo" params="is_ign sensors_params_file">
+    <xacro:read_sensor_config_data qcar_sensors_params_file="${sensors_params_file}"/>
     <xacro:property name="max_steering_angle" value="0.3"/>
     <xacro:property name="axle_vel_limit" value="244.8696"/>
@@ -18,5 +19,5 @@
       <sensor type="camera" name="intelrealsense_rgb">
         <always_on>1</always_on>
-        <update_rate>60.0</update_rate>
+        <update_rate>${rgb_update_rate}</update_rate>
         <visualize>true</visualize>
         <topic>qcar/rgb/image_raw</topic>
@@ -24,11 +25,11 @@
           <horizontal_fov>1.21126</horizontal_fov>
           <image>
-              <width>640</width>
-              <height>480</height>
-              <format>R8G8B8</format>
-          </image>
-          <clip>
-              <near>0.02</near>
-              <far>300</far>
+              <width>${rgbd_width}</width>
+              <height>${rgbd_height}</height>
+              <format>R8G8B8</format>
+          </image>
+          <clip>
+              <near>${rgbd_clip_near}</near>
+              <far>${rgbd_clip_far}</far>
           </clip>
           <noise>
@@ -63,5 +64,5 @@
       <sensor type="camera" name="csi_front">
         <always_on>1</always_on>
-        <update_rate>60.0</update_rate>
+        <update_rate>${csi_update_rate}</update_rate>
         <visualize>true</visualize>
         <topic>qcar/csi_front/image_raw</topic>
@@ -69,11 +70,11 @@
           <horizontal_fov>2.79253</horizontal_fov>
           <image>
-              <width>1280</width>
-              <height>640</height>
-              <format>R8G8B8</format>
-          </image>
-          <clip>
-              <near>0.02</near>
-              <far>300</far>
+              <width>${csi_width}</width>
+              <height>${csi_height}</height>
+              <format>R8G8B8</format>
+          </image>
+          <clip>
+              <near>${csi_clip_near}</near>
+              <far>${csi_clip_far}</far>
           </clip>
           <noise>
@@ -108,5 +109,5 @@
       <sensor type="camera" name="csi_right">
         <always_on>1</always_on>
-        <update_rate>60.0</update_rate>
+        <update_rate>${csi_update_rate}</update_rate>
         <visualize>true</visualize>
         <topic>qcar/csi_right/image_raw</topic>
@@ -114,11 +115,11 @@
           <horizontal_fov>2.79253</horizontal_fov>
           <image>
-              <width>1280</width>
-              <height>640</height>
-              <format>R8G8B8</format>
-          </image>
-          <clip>
-              <near>0.02</near>
-              <far>300</far>
+              <width>${csi_width}</width>
+              <height>${csi_height}</height>
+              <format>R8G8B8</format>
+          </image>
+          <clip>
+              <near>${csi_clip_near}</near>
+              <far>${csi_clip_far}</far>
           </clip>
           <noise>
@@ -153,5 +154,5 @@
       <sensor type="camera" name="csi_left">
         <always_on>1</always_on>
-        <update_rate>60.0</update_rate>
+        <update_rate>${csi_update_rate}</update_rate>
         <visualize>true</visualize>
         <topic>qcar/csi_left/image_raw</topic>
@@ -159,11 +160,11 @@
           <horizontal_fov>2.79253</horizontal_fov>
           <image>
-              <width>1280</width>
-              <height>640</height>
-              <format>R8G8B8</format>
-          </image>
-          <clip>
-              <near>0.02</near>
-              <far>300</far>
+              <width>${csi_width}</width>
+              <height>${csi_height}</height>
+              <format>R8G8B8</format>
+          </image>
+          <clip>
+              <near>${csi_clip_near}</near>
+              <far>${csi_clip_far}</far>
           </clip>
           <noise>
@@ -198,5 +199,5 @@
       <sensor type="camera" name="csi_back">
         <always_on>1</always_on>
-        <update_rate>60.0</update_rate>
+        <update_rate>${csi_update_rate}</update_rate>
         <visualize>true</visualize>
         <topic>qcar/csi_back/image_raw</topic>
@@ -204,11 +205,11 @@
           <horizontal_fov>2.79253</horizontal_fov>
           <image>
-              <width>1280</width>
-              <height>640</height>
-              <format>R8G8B8</format>
-          </image>
-          <clip>
-              <near>0.02</near>
-              <far>300</far>
+              <width>${csi_width}</width>
+              <height>${csi_height}</height>
+              <format>R8G8B8</format>
+          </image>
+          <clip>
+              <near>${csi_clip_near}</near>
+              <far>${csi_clip_far}</far>
           </clip>
           <noise>
@@ -233,7 +234,7 @@
       <sensor type="gpu_lidar" name="rplidar_a2m8">
         <always_on>true</always_on>
-        <pose>0 0 0 0 0 0</pose>
-        <visualize>true</visualize>
-        <update_rate>10</update_rate>
+        <pose>0 0 0.0114 0 0 0</pose>
+        <visualize>true</visualize>
+        <update_rate>${lidar_update_rate}</update_rate>
         <topic>scan</topic>
         <gz_frame_id>lidar</gz_frame_id>
@@ -241,5 +242,5 @@
             <scan>
                 <horizontal>
-                    <samples>800</samples>
+                    <samples>${lidar_num_points}</samples>
                     <resolution>1</resolution>
                     <!-- <min_angle>-1.570796</min_angle>
@@ -250,6 +251,6 @@
             </scan>
             <range>
-                <min>0.20</min>
-                <max>12.0</max>
+                <min>${lidar_min_range}</min>
+                <max>${lidar_max_range}</max>
                 <resolution>0.01</resolution>
             </range>
@@ -269,5 +270,5 @@
       <sensor name="imu" type="imu">
         <always_on>1</always_on>
-        <update_rate>60.0</update_rate>
+        <update_rate>${imu_update_rate}</update_rate>
         <visualize>true</visualize>
         <topic>imu</topic>

File: qcar_description/urdf/qcar.materials.xacro (robot description, xacro)
@@ -25,3 +25,33 @@
     <color rgba="1.0 1.0 1.0 1.0"/>
   </material>
+  <xacro:macro name="read_sensor_config_data" params="qcar_sensors_params_file">
+      <!-- Read .yaml files from disk, load content into properties -->
+      <xacro:property name="config_sensors_parameters" value="${xacro.load_yaml(qcar_sensors_params_file)}"/>
+      <!-- Extract subsections from yaml dictionaries -->
+      <xacro:property name="csi_properties" value="${config_sensors_parameters['sensors_parameters']['csi_camera']}"/>
+      <xacro:property name="rgbd_properties" value="${config_sensors_parameters['sensors_parameters']['rgbd_camera']}"/>
+      <xacro:property name="imu_properties" value="${config_sensors_parameters['sensors_parameters']['imu']}"/>
+      <xacro:property name="lidar_properties" value="${config_sensors_parameters['sensors_parameters']['lidar']}"/>
+      <!-- Sensors Properties -->
+      <!-- CSI -->
+      <xacro:property name="csi_update_rate" value="${csi_properties['update_rate']}" scope="parent"/>
+      <xacro:property name="csi_width" value="${csi_properties['image_width']}" scope="parent"/>
+      <xacro:property name="csi_height" value="${csi_properties['image_height']}" scope="parent"/>
+      <xacro:property name="csi_clip_near" value="${csi_properties['clip_near']}" scope="parent"/>
+      <xacro:property name="csi_clip_far" value="${csi_properties['clip_far']}" scope="parent"/>
+      <!-- RGBD -->
+      <xacro:property name="rgb_update_rate" value="${rgbd_properties['rgb_update_rate']}" scope="parent"/>
+      <xacro:property name="depth_update_rate" value="${rgbd_properties['depth_update_rate']}" scope="parent"/>
+      <xacro:property name="rgbd_width" value="${rgbd_properties['image_width']}" scope="parent"/>
+      <xacro:property name="rgbd_height" value="${rgbd_properties['image_height']}" scope="parent"/>
+      <xacro:property name="rgbd_clip_near" value="${rgbd_properties['clip_near']}" scope="parent"/>
+      <xacro:property name="rgbd_clip_far" value="${rgbd_properties['clip_far']}" scope="parent"/>
+      <!-- IMU -->
+      <xacro:property name="imu_update_rate" value="${imu_properties['update_rate']}" scope="parent"/>
+      <!-- LIDAR -->
+      <xacro:property name="lidar_update_rate" value="${lidar_properties['update_rate']}" scope="parent"/>
+      <xacro:property name="lidar_num_points" value="${lidar_properties['num_points']}" scope="parent"/>
+      <xacro:property name="lidar_max_range" value="${lidar_properties['max_range']}" scope="parent"/>
+      <xacro:property name="lidar_min_range" value="${lidar_properties['min_range']}" scope="parent"/>
+  </xacro:macro>
 </robot>

File: qcar_description/urdf/qcar_ros2.urdf.xacro (robot description, xacro)
@@ -32,5 +32,4 @@
     <!-- includes -->
     <!-- <xacro:include filename="$(find qcar_description)/urdf/qcar.gazebo.xacro" /> -->
-    <xacro:include filename="$(find qcar_description)/urdf/qcar.materials.xacro" />
     <!-- Degree-to-radian conversions -->
     <xacro:property name="degrees_30" value="0.523599"/>

File: qcar_description/urdf/qcar_system.urdf.xacro (robot description, xacro)
@@ -7,4 +7,6 @@
   <xacro:arg name="is_ign" default="false" />
   <xacro:arg name="prefix" default="" />
+  <xacro:arg name="sensors_params_file" default="$(find qcar_description)/config/sensor_params.yaml"/>
+  <xacro:include filename="$(find qcar_description)/urdf/qcar.materials.xacro" />
   <xacro:include filename="$(find qcar_description)/urdf/qcar_ros2.urdf.xacro" />
   <!-- Import all Gazebo-customization elements, including Gazebo colors -->
@@ -22,5 +24,5 @@
     <origin xyz="0 0 0" rpy="0 0 0" />
   </xacro:QCar>
-  <xacro:qcar_gazebo is_ign="$(arg is_ign)"/>
+  <xacro:qcar_gazebo is_ign="$(arg is_ign)" sensors_params_file="$(arg sensors_params_file)"/>
   <!-- <xacro:QCar_control name="QCar" prefix="$(arg prefix)"/> -->
 </robot>
