Commit message: modification:  found better friction parameters for qcar gazebo, works better but I am not fully convinced

File: ackermann_vehicle_description/urdf/mobile_base_gazebo.xacro (robot description, xacro)
@@ -7,18 +7,82 @@
   </gazebo>
   <gazebo reference="front_right_wheel_link">
-    <mu1>10.0</mu1>
-    <mu2>10.0</mu2>
+    <collision>
+      <surface>
+        <friction>
+          <ode>
+            <mu>0.90000000000000002</mu>
+            <mu2>0.90000000000000002</mu2>
+            <slip1>0</slip1>
+            <slip2>0</slip2>
+          </ode>
+        </friction>
+        <contact>
+          <ode>
+            <kp>1000000000</kp>
+            <min_depth>0.001</min_depth>
+          </ode>
+        </contact>
+      </surface>
+    </collision>
   </gazebo>
   <gazebo reference="front_left_wheel_link">
-    <mu1>10.0</mu1>
-    <mu2>10.0</mu2>
+    <collision>
+      <surface>
+        <friction>
+          <ode>
+            <mu>0.90000000000000002</mu>
+            <mu2>0.90000000000000002</mu2>
+            <slip1>0</slip1>
+            <slip2>0</slip2>
+          </ode>
+        </friction>
+        <contact>
+          <ode>
+            <kp>1000000000</kp>
+            <min_depth>0.001</min_depth>
+          </ode>
+        </contact>
+      </surface>
+    </collision>
   </gazebo>
   <gazebo reference="rear_right_wheel_link">
-    <mu1>10.0</mu1>
-    <mu2>10.0</mu2>
+    <collision>
+      <surface>
+        <friction>
+          <ode>
+            <mu>1.1000000000000001</mu>
+            <mu2>1.1000000000000001</mu2>
+            <slip1>0</slip1>
+            <slip2>0</slip2>
+          </ode>
+        </friction>
+        <contact>
+          <ode>
+            <kp>1000000000</kp>
+            <min_depth>0.001</min_depth>
+          </ode>
+        </contact>
+      </surface>
+    </collision>
   </gazebo>
   <gazebo reference="rear_left_wheel_link">
-    <mu1>10.0</mu1>
-    <mu2>10.0</mu2>
+    <collision>
+      <surface>
+        <friction>
+          <ode>
+            <mu>1.1000000000000001</mu>
+            <mu2>1.1000000000000001</mu2>
+            <slip1>0</slip1>
+            <slip2>0</slip2>
+          </ode>
+        </friction>
+        <contact>
+          <ode>
+            <kp>1000000000</kp>
+            <min_depth>0.001</min_depth>
+          </ode>
+        </contact>
+      </surface>
+    </collision>
   </gazebo>
   <!-- Gazebo Plugins -->

File: qcar_description/urdf/qcar.gazebo.xacro (robot description, xacro)
@@ -339,6 +339,12 @@
       </joint>
       <joint name="right_steering_joint">
-        <param name="mimic">left_steering_joint</param> <!-- Command this joint -->
-        <param name="multiplier">1</param> <!-- Move in the opposite direction -->
+        <command_interface name="position">
+          <param name="min">${-max_steering_angle}</param>
+          <param name="max">${max_steering_angle}</param>
+        </command_interface>
+        <!-- Command this joint -->
+        <!-- <param name="mimic">left_steering_joint</param>  -->
+        <!-- Move in the opposite direction -->
+        <!-- <param name="multiplier">1</param>  -->
         <state_interface name="position"/>
         <state_interface name="velocity"/>
@@ -346,8 +352,10 @@
       </joint>
       <joint name="right_front_axle">
-        <command_interface name="velocity">
+        <param name="mimic">right_rear_axle</param>
+        <param name="multiplier">1</param>
+        <!-- <command_interface name="velocity">
           <param name="min">${-axle_vel_limit}</param>
           <param name="max">${axle_vel_limit}</param>
-        </command_interface>
+        </command_interface> -->
         <state_interface name="position"/>
         <state_interface name="velocity"/>
@@ -355,6 +363,10 @@
       </joint>
       <joint name="left_front_axle">
-        <param name="mimic">right_front_axle</param> <!-- Command this joint -->
-        <param name="multiplier">-1</param> <!-- Move in the opposite direction -->
+        <param name="mimic">left_rear_axle</param>
+        <param name="multiplier">1</param>
+        <!-- <command_interface name="velocity">
+          <param name="min">${-axle_vel_limit}</param>
+          <param name="max">${axle_vel_limit}</param>
+        </command_interface> -->
         <state_interface name="position"/>
         <state_interface name="velocity"/>

File: qcar_description/urdf/qcar_ros2.urdf.xacro (robot description, xacro)
@@ -296,6 +296,6 @@
       <child link="left_front_axle_carrier"/>
       <axis xyz = "0 0 1"/>
-      <!-- <limit lower="-0.523599" upper="0.523599" effort="0.5649" velocity="4.553"/> -->
-      <limit lower="-0.3" upper="0.3" effort="0.5649" velocity="4.553"/>
+      <limit lower="-0.523599" upper="0.523599" effort="0.5649" velocity="4.553"/>
+      <!-- <limit lower="-0.3" upper="0.3" effort="0.5649" velocity="4.553"/> -->
     </joint>
     <link name="left_front_axle_carrier">
@@ -305,9 +305,9 @@
       <parent link="left_front_axle_carrier"/>
       <child link="left_front_wheel"/>
-      <axis xyz="0 1 0"/>
+      <axis xyz="0 -1 0"/>
       <origin rpy="0 0 3.14159"/>
       <limit effort="5.12766" velocity="244.8696"/>
       <dynamics damping="0.1" friction="0.1"/>
-      <mimic joint="right_front_axle" multiplier="-1.0" offset="0"/>
+      <mimic joint="left_rear_axle" multiplier="1.0" offset="0"/>
     </joint>
     <transmission name="left_front_axle_trans">
@@ -329,6 +329,8 @@
       </visual>
       <collision>
-        <origin rpy="0 0 0" xyz="0 0 0"/>
-        <geometry>
+        <!-- <origin rpy="0 0 0" xyz="0 -0.0225 0"/> -->
+        <origin rpy="0 0 0" xyz="0 0 0"/>
+        <geometry>
+          <!-- <sphere radius="0.034"/> -->
     <mesh filename="file://$(find qcar_description)/meshes/QCarWheel.stl" scale="0.001 0.001 0.001"/>
         </geometry>
@@ -356,5 +358,7 @@
       <axis xyz="0 1 0"/>
       <!--<limit effort="${axle_eff_limit}" velocity="${axle_vel_limit}"/>-->
+      <limit effort="5.12766" velocity="244.8696"/>
       <dynamics damping="0.1" friction="0.1"/>
+      <mimic joint="right_rear_axle" multiplier="1.0" offset="0"/>
     </joint>
     <transmission name="right_front_axle_trans">
@@ -376,6 +380,8 @@
       </visual>
       <collision>
-        <origin rpy="0 0 0" xyz="0 0 0"/>
-        <geometry>
+        <!-- <origin rpy="0 0 0" xyz="0 -0.0225 0"/> -->
+        <origin rpy="0 0 0" xyz="0 0 0"/>
+        <geometry>
+          <!-- <sphere radius="0.034"/> -->
     <mesh filename="file://$(find qcar_description)/meshes/QCarWheel.stl" scale="0.001 0.001 0.001"/>
         </geometry>
@@ -410,7 +416,7 @@
       <child link="right_front_axle_carrier"/>
       <axis xyz = "0 0 1"/>
-      <!-- <limit lower="0.523599" upper="0.523599" effort="0.5649" velocity="4.553"/> -->
-      <limit lower="-0.3" upper="0.3" effort="0.5649" velocity="4.553"/>
-      <mimic joint="left_steering_joint" multiplier="1.0" offset="0"/>
+      <limit lower="-0.523599" upper="0.523599" effort="0.5649" velocity="4.553"/>
+      <!-- <limit lower="-0.3" upper="0.3" effort="0.5649" velocity="4.553"/> -->
+      <!-- <mimic joint="left_steering_joint" multiplier="1.0" offset="0"/> -->
     </joint>
     <transmission name="right_steering_trans">
@@ -455,6 +461,8 @@
       </visual>
       <collision>
-        <origin rpy="0 0 0" xyz="0 0 0"/>
-        <geometry>
+        <!-- <origin rpy="0 0 0" xyz="0 -0.0225 0"/> -->
+        <origin rpy="0 0 0" xyz="0 0 0"/>
+        <geometry>
+          <!-- <sphere radius="0.034"/> -->
     <mesh filename="file://$(find qcar_description)/meshes/QCarWheel.stl" scale="0.001 0.001 0.001"/>
         </geometry>
@@ -498,6 +506,8 @@
       </visual>
       <collision>
-        <origin rpy="0 0 0" xyz="0 0 0"/>
-        <geometry>
+        <!-- <origin rpy="0 0 0" xyz="0 -0.0225 0"/> -->
+        <origin rpy="0 0 0" xyz="0 0 0"/>
+        <geometry>
+          <!-- <sphere radius="0.034"/> -->
     <mesh filename="file://$(find qcar_description)/meshes/QCarWheel.stl" scale="0.001 0.001 0.001"/>
         </geometry>
@@ -523,14 +533,13 @@
           <friction>
             <ode>
-              <mu>1.0</mu>
-              <mu2>1.0</mu2>
-              <fdir1>0 0 1</fdir1>
+              <mu>1.0000000000000002</mu>
+              <mu2>1.0000000000000002</mu2>
+              <slip1>0</slip1>
+              <slip2>0</slip2>
             </ode>
           </friction>
           <contact>
             <ode>
-              <kp>1000000.0</kp>
-              <kd>100.0</kd>
-              <max_vel>0.1</max_vel>
+              <kp>1000000000</kp>
               <min_depth>0.001</min_depth>
             </ode>
@@ -544,14 +553,13 @@
           <friction>
             <ode>
-              <mu>1.0</mu>
-              <mu2>1.0</mu2>
-              <fdir1>0 0 1</fdir1>
+              <mu>1.0000000000000002</mu>
+              <mu2>1.0000000000000002</mu2>
+              <slip1>0</slip1>
+              <slip2>0</slip2>
             </ode>
           </friction>
           <contact>
             <ode>
-              <kp>1000000.0</kp>
-              <kd>100.0</kd>
-              <max_vel>0.1</max_vel>
+              <kp>1000000000</kp>
               <min_depth>0.001</min_depth>
             </ode>
@@ -565,14 +573,13 @@
           <friction>
             <ode>
-              <mu>1.0</mu>
-              <mu2>1.0</mu2>
-              <fdir1>0 0 1</fdir1>
+              <mu>1.1000000000000001</mu>
+              <mu2>1.1000000000000001</mu2>
+              <slip1>0</slip1>
+              <slip2>0</slip2>
             </ode>
           </friction>
           <contact>
             <ode>
-              <kp>1000000.0</kp>
-              <kd>100.0</kd>
-              <max_vel>0.1</max_vel>
+              <kp>1000000000</kp>
               <min_depth>0.001</min_depth>
             </ode>
@@ -586,14 +593,13 @@
           <friction>
             <ode>
-              <mu>1.0</mu>
-              <mu2>1.0</mu2>
-              <fdir1>0 0 1</fdir1>
+              <mu>1.1000000000000001</mu>
+              <mu2>1.1000000000000001</mu2>
+              <slip1>0</slip1>
+              <slip2>0</slip2>
             </ode>
           </friction>
           <contact>
             <ode>
-              <kp>1000000.0</kp>
-              <kd>100.0</kd>
-              <max_vel>0.1</max_vel>
+              <kp>1000000000</kp>
               <min_depth>0.001</min_depth>
             </ode>
