Commit message: 🚀 Autonomous Racing v13.0 — Vision-Fused Intelligent Racing Edition
Highlights:
- **Active Lane-Assist (v13)**: Integrated a new Computer Vision layer using OpenCV for real-time lane center estimation (Yellow/White line detection).
- **Vision-Control Fusion**: The navigator now combines Pure Pursuit (Global Path) + APF (Local Obstacles) + Lane-Assist (Visual alignment) for a 3-layer autonomous control.
- **Sensor Calibration**: Major overhaul of the URDF camera configurations (FOV fix, pitch adjustment, and lateral symmetry) for distortion-free computer vision.
- **Node Expansion**: Added 'lane_detector.py' and updated 'telemetry_dashboard' with Vision HUD (confidence badges and offset bar).
- **Documentation**: Updated README with mathematical formalisms for the vision pipeline and revised Phase 4 roadmap.

File: src/roboracer/roboracer_description/urdf/qcar.gazebo.xacro (robot description, xacro)
@@ -68,5 +68,5 @@
         <topic>qcar/csi_front/image_raw</topic>
         <camera name="front">
-          <horizontal_fov>2.79253</horizontal_fov>
+          <horizontal_fov>1.22</horizontal_fov>
           <image>
               <width>${csi_width}</width>
@@ -113,5 +113,5 @@
         <topic>qcar/csi_right/image_raw</topic>
         <camera name="right">
-          <horizontal_fov>2.79253</horizontal_fov>
+          <horizontal_fov>1.40</horizontal_fov>
           <image>
               <width>${csi_width}</width>
@@ -157,6 +157,6 @@
         <visualize>true</visualize>
         <topic>qcar/csi_left/image_raw</topic>
-        <camera name="front">
-          <horizontal_fov>2.79253</horizontal_fov>
+        <camera name="left">
+          <horizontal_fov>1.40</horizontal_fov>
           <image>
               <width>${csi_width}</width>
@@ -202,6 +202,6 @@
         <visualize>true</visualize>
         <topic>qcar/csi_back/image_raw</topic>
-        <camera name="front">
-          <horizontal_fov>2.79253</horizontal_fov>
+        <camera name="back">
+          <horizontal_fov>1.50</horizontal_fov>
           <image>
               <width>${csi_width}</width>

File: src/roboracer/roboracer_description/urdf/qcar_ros2.urdf.xacro (robot description, xacro)
@@ -199,17 +199,14 @@
     </link>
     <joint name="camera_rgb_joint" type="fixed">
-      <!-- <axis xyz="0 1 0" /> -->
-      <!-- <origin xyz=".2 0 0" rpy="0 0 0"/> -->
-        <origin rpy="0 0 0" xyz="0.081686 0.031547 0.15445"/>
-        <!-- <origin rpy="0 0 0" xyz="0 0 0"/> -->
-      <parent link="base"/>
-      <child link="camera_rgb"/>
+        <!-- RealSense RGB: centrada en Y, sobre el techo (z=0.154). -->
+        <origin rpy="0 0 0" xyz="0.081686 0.0 0.15445"/>
+        <parent link="base"/>
+        <child link="camera_rgb"/>
     </joint>
     <link name="camera_rgb"/>
     <joint name="camera_csi_front_joint" type="fixed">
-        <!-- <axis xyz="0 1 0" /> -->
-        <!-- <origin xyz=".2 0 0" rpy="0 0 0"/> -->
-        <origin rpy="0 0 0" xyz="0.19236 -0.000475 0.093029"/>
-        <!-- <origin rpy="0 0 0" xyz="0 0 0"/> -->
+        <!-- Cámara frontal: centrada lateralmente (y=0), ligeramente inclinada
+             hacia abajo (pitch 0.15 rad ≈ 8.6°) para ver mejor el asfalto. -->
+        <origin rpy="0 0.15 0" xyz="0.19236 0.0 0.093029"/>
         <parent link="base"/>
         <child link="camera_csi_front"/>
@@ -217,10 +214,6 @@
     <link name="camera_csi_front"/>
     <joint name="camera_csi_right_joint" type="fixed">
-        <!-- <axis xyz="0 1 0" /> -->
-        <!-- <origin xyz=".2 0 0" rpy="0 0 0"/> -->
-        <!-- ___________________xyz is wrong, need to update_______________________________ -->
-        <!-- <origin rpy="0 0 -1.5708" xyz="0.12887 -0.06755 0.093029"/> -->
-        <origin rpy="0 0 -1.5708" xyz="0.012887 -0.06755 0.093029"/>
-        <!-- <origin rpy="0 0 0" xyz="0 0 0"/> -->
+        <!-- Cámara lateral DERECHA: rotada -90° en Z, en el costado derecho (y=-0.06). -->
+        <origin rpy="0 0 -1.5708" xyz="0.01289 -0.06000 0.093029"/>
         <parent link="base"/>
         <child link="camera_csi_right"/>
@@ -228,8 +221,6 @@
     <link name="camera_csi_right"/>
     <joint name="camera_csi_back_joint" type="fixed">
-        <!-- <axis xyz="0 1 0" /> -->
-        <!-- <origin xyz=".2 0 0" rpy="0 0 0"/> -->
-        <origin rpy="0 0 -3.1416" xyz="-0.16669 -0.000578 0.093029"/>
-        <!-- <origin rpy="0 0 0" xyz="0 0 0"/> -->
+        <!-- Cámara trasera: rotada 180° en Z (mira hacia atrás), centrada en Y. -->
+        <origin rpy="0 0 -3.1416" xyz="-0.16669 0.0 0.093029"/>
         <parent link="base"/>
         <child link="camera_csi_back"/>
@@ -237,10 +228,6 @@
     <link name="camera_csi_back"/>
     <joint name="camera_csi_left_joint" type="fixed">
-        <!-- <axis xyz="0 1 0" /> -->
-        <!-- <origin xyz=".2 0 0" rpy="0 0 0"/> -->
-        <!-- ___________________xyz is wrong, need to update_______________________________ -->
-        <!-- <origin rpy="0 0 1.5708" xyz="0.12784 0.052497 0.093029"/> -->
-         <origin rpy="0 0 1.5708" xyz="0.012784 0.052497 0.093029"/>
-        <!-- <origin rpy="0 0 0" xyz="0 0 0"/> -->
+        <!-- Cámara lateral IZQUIERDA: rotada +90° en Z, espejo de la derecha (y=+0.06). -->
+        <origin rpy="0 0 1.5708" xyz="0.01289 0.06000 0.093029"/>
         <parent link="base"/>
         <child link="camera_csi_left"/>
